File: Kicad/makeraxe-lite.kicad_pcb (KiCad board)
At the start: 2 copper layers, 56.5 x 99.8 mm, 142 parts, among them IC1 CH224K, J1 Conn_01x02, J2 USB_C_Receptacle_USB2.0, J3 TC2030-IDC, J4 Conn_01x04, J5 USB_C_Receptacle_USB2.0, J6 Conn_01x04, Q1 2N7002K, Q2 CSD17311Q5, Q3 CSD17311Q5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

Commit message: V0.35 Release
Parts:
- removed C10: 0.47uF, Capacitor_SMD:C_0805_2012Metric
- removed C11: 22uF, Capacitor_SMD:C_0805_2012Metric
- removed the REF** at (115.6, 142.7)
- added C52: 0.47uF, bitaxe:T491A, B.Cu at (105.8, 52.6)
- added C53: 22uF, bitaxe:T495C, B.Cu at (111.2, 52.6)
- added REF**: OSHW-Logo2_14.6x12mm_SilkScreen, Symbol:OSHW-Logo2_14.6x12mm_SilkScreen, B.Cu at (116.1, 141.6)
- R10: value 0 -> 24K; moved to F.Cu
- U3: footprint bitaxe:SOT230P700X180-4N -> Package_TO_SOT_SMD:TO-263-3_TabPin2
- moved R10 25.7 mm to (92.9, 49.7), turned to 90 degrees
- moved U3 8.32 mm to (113.1, 53.3), turned to 0 degrees
- moved R3 1.55 mm to (92.9, 48.2)
Connections:
- IC1 pad 9: unconnected-(IC1-CFG1-Pad9) -> Net-(IC1-CFG1)
- R10 pad 1: /ESP32/PLUG_SENSE -> GND
- R10 pad 2: GND -> Net-(IC1-CFG1)
Routing:
- net /5V: track 200.7 -> 195.7 mm, vias 11 -> 10
- net Net-(IC1-CFG1): track 0.00 -> 4.40 mm
- net /Power/Vin_20V: track 77.6 -> 80.9 mm, vias 19 -> 21
- net /ESP32/PLUG_SENSE: track 10.6 -> 7.44 mm
- net Net-(IC1-VBUS): track 3.30 -> 4.82 mm
- net GND: track 323.6 -> 322.2 mm, vias 84 -> 108
- net /ESP32/IO0: track 96.4 -> 95.7 mm
- net /VDD: track 71.6 -> 71.0 mm
Other:
- board text added: "12V/20W"
- board text added: "USB PD"
- board text added: "V035"
- board text added: "https://makingdevices.com/miners"
- board text removed: "Power"
- board text removed: "V025"
- board text removed: "https://makingdevices.com/links"
