File: Kicad/power.kicad_sch (KiCad schematic)
At the start: 40 parts, among them IC1 CH224K, J1 Conn_01x02, J2 USB_C_Receptacle_USB2.0, Q1 2N7002K, Q2 CSD17311Q5, Q3 CSD17311Q5, U2 INA260, U3 TS2940CW55_RPG, U4 TPS40305, U5 DS4432U+

Commit message: V0.35 Release
Parts:
- removed C10: 0.47uF, Capacitor_SMD:C_0805_2012Metric, symbol Device:C
- removed C11: 22uF, Capacitor_SMD:C_0805_2012Metric, symbol Device:C
- added C52: 0.47uF, bitaxe:T491A, symbol bitaxe:T491A474K025AT7280
- added C53: 22uF, bitaxe:T495C, symbol bitaxe:T495C226K025ATE300
- added R10: 24K, Resistor_SMD:R_0402_1005Metric, symbol Device:R_US
- U3: footprint SOT230P700X180-4N -> Package_TO_SOT_SMD:TO-263-3_TabPin2
Connections:
- net 5V: now also C53.1 (+)
- net GND: now also C52.2 (-), C53.2 (-), R10.1
- net Vin_20V: now also C52.1 (+)
- net at IC1.9 (CFG1): now also R10.2
- no-connect marks 9 -> 8
Other:
- moved on the sheet: R3
